File: led_cubic.kicad_sch (KiCad schematic)
At the start: 130 parts, among them J1 Cathode Layer, Q1 2N2222, Q2 2N2222, Q3 2N2222, Q4 2N2222, U1 74HC595, U2 74HC595, U3 74HC595, U4 74HC595, U5 74HC595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

Commit message: 0.1.1
修改布局和PCB大小并添加M3螺丝孔
Parts:
- J1: footprint Connector_PinSocket_2.54mm:PinSocket_1x04_P2.54mm_Vertical -> Library:PinSocket_1x04_P2.54mm_Vertical
- U1, U2, U3, U4, U5, U6, U7: footprint Package_DIP:DIP-16_W7.62mm_Socket -> Library:DIP-16_W7.62mm_Socket
Other:
- moved on the sheet: D1, D10, D11, D12, D13, D14, D15, D16, D17, D18, D19, D2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
